File: compaq_lte_expanded_memory.kicad_sch (KiCad schematic)
At the start: 17 parts, among them J1 Conn_02x30_Odd_Even, U1 DRAM-1Mx4-SOJ-24, U10 DRAM-1Mx4-SOJ-24, U11 DRAM-1Mx4-SOJ-24, U12 DRAM-1Mx4-SOJ-24, U13 DRAM-1Mx4-SOJ-24, U14 DRAM-1Mx4-SOJ-24, U15 DRAM-1Mx4-SOJ-24, U16 DRAM-1Mx4-SOJ-24, U2 DRAM-1Mx4-SOJ-24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

Commit message: latest before moving to original Compaq module
Parts:
- added R1, R2, R3: 330, Resistor_SMD:R_0805_2012Metric, symbol Device:R
Connections:
- net +5V: now also R1.1, R2.1, R3.1
- net CFG_1_?: now also R1.2
- net CFG_2_?: now also R2.2
- net ~{RAS2}: now also J1.10 (Pin_10), U10.4 (~{RAS}), U12.4 (~{RAS}), U14.4 (~{RAS}), U16.4 (~{RAS}); no longer J1.57 (Pin_57), U1.4 (~{RAS}), U3.4 (~{RAS}), U5.4 (~{RAS}), U7.4 (~{RAS})
- net ~{RAS3}: now also J1.57 (Pin_57), U1.4 (~{RAS}), U3.4 (~{RAS}), U5.4 (~{RAS}), U7.4 (~{RAS}); no longer J1.58 (Pin_58), U2.4 (~{RAS}), U4.4 (~{RAS}), U6.4 (~{RAS}), U8.4 (~{RAS})
- net ~{RAS4}: now also J1.58 (Pin_58), U2.4 (~{RAS}), U4.4 (~{RAS}), U6.4 (~{RAS}), U8.4 (~{RAS}); no longer J1.10 (Pin_10), U10.4 (~{RAS}), U12.4 (~{RAS}), U14.4 (~{RAS}), U16.4 (~{RAS})
- net ~{RASY} renamed ~{RAS1}
- net ~{WE2} renamed ~{WE}
Other:
- moved on the sheet: J1, U1, U10, U11, U12, U13, U14, U15, U16, U2, U3, U4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
